File: Hardware/MCU_STM32F412RGT6_0x00.kicad_sch (KiCad schematic)
At the start: 68 parts, among them J1 USB4105-GF-A, J10 Conn_01x02, J11 Conn_01x02, J2 Conn_01x04, J3 Conn_01x04, J4 Conn_01x04, J5 Conn_01x03, J6 Conn_01x04, J7 Conn_01x06, J8 Conn_01x02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

Commit message: Final layout for V1, sent of to FAB
Parts:
- removed C14: 100n, Capacitor_SMD:C_0805_2012Metric_Pad1.18x1.45mm_HandSolder, symbol Device:C_Small
- removed D1, D2, D3: LED, LED_SMD:LED_PLCC-2, symbol Device:LED
- removed R2, R3, R4, R5, R6: 10k, Resistor_SMD:R_0805_2012Metric_Pad1.20x1.40mm_HandSolder, symbol Device:R_Small
- removed U3: MS5611-01BA, Package_LGA:LGA-8_3x5mm_P1.25mm, symbol Sensor_Pressure:MS5611-01BA
- gave numbers to parts that had none: 3
Connections:
- net CAN_RX: now also J4.2 (Pin_2), U9.4; no longer J4.3 (Pin_3), U9.3
- net CAN_TX: now also J4.3 (Pin_3), U9.3; no longer J4.2 (Pin_2), U9.4
- net SCL: now also J2.2 (Pin_2), U7.4; no longer J2.3 (Pin_3), U7.3
- net SDA: now also J2.3 (Pin_3), U7.3; no longer J2.2 (Pin_2), U7.4
- net SWDCLK: now also J6.2 (Pin_2), U5.4; no longer J6.3 (Pin_3), U5.3
- net SWDIO: now also J6.3 (Pin_3), U5.3; no longer J6.2 (Pin_2), U5.4
Other:
- note added: "CAN"
- note added: "Crystal"
- note added: "I2C"
- note added: "I2S"
- note added: "MCU"
- note added: "MECH"
- note added: "SWD"
- note added: "UART"
- moved on the sheet: C1, C10, C11, C12, C13, C2, C3, C4, C5, C6, C7, C8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
