File: Hardware/universal.kicad_pcb (KiCad board)
At the start: 2 copper layers, 50.8 x 39.4 mm, 76 parts, among them J1 USB_B_Mini, J2 Conn_01x04, J3 Conn_01x04, J4 Conn_01x04, J5 Conn_01x03, J6 Conn_01x04, U1 STM32F412RGTx, U2 NUP4202, U3 MS5611-01BA, Y1 Crystal_GND24_Small

Commit message: new usb connector and pcb size defined
Parts:
- removed JP1: SolderJumper_3_Open, Jumper:SolderJumper-3_P1.3mm_Open_Pad1.0x1.5mm
- removed PA0, PA1, PA10, PA2, PA3, PA4, PA5, PA6, PA7, PA8, PA9, PB0, PB1, PB12, PB13, PB14, PB15, PB2, PB3, PB4, PB5, PC0, PC1, PC10, PC11, PC12, PC13, PC14, PC15, PC2, PC3, PC4, PC6, PC7, PC8, PC9: TestPoint, TestPoint:TestPoint_Pad_D1.5mm
- added C15: 100pF, Capacitor_SMD:C_0805_2012Metric_Pad1.18x1.45mm_HandSolder, F.Cu at (167.9, 99.8)
- added C16: 100pF, Capacitor_SMD:C_0805_2012Metric_Pad1.18x1.45mm_HandSolder, F.Cu at (160.5, 97.5)
- added C17: 100pF, Capacitor_SMD:C_0805_2012Metric_Pad1.18x1.45mm_HandSolder, F.Cu at (174.5, 95.0)
- added C18: 100pF, Capacitor_SMD:C_0805_2012Metric_Pad1.18x1.45mm_HandSolder, F.Cu at (172.0, 90.9)
- added C9: 100nF, Capacitor_SMD:C_0805_2012Metric_Pad1.18x1.45mm_HandSolder, F.Cu at (143.8, 86.9)
- added D4: LED, LED_SMD:LED_PLCC-2, F.Cu at (131.2, 80.9)
- added D5: BAV99, Package_TO_SOT_SMD:SOT-23, F.Cu at (167.5, 94.3)
- added D6: BAV99, Package_TO_SOT_SMD:SOT-23, F.Cu at (175.3, 97.8)
- added D7: BAV99, Package_TO_SOT_SMD:SOT-23, F.Cu at (175.3, 89.9)
- added D8: BAV99, Package_TO_SOT_SMD:SOT-23, F.Cu at (164.8, 99.8)
- added J10: Conn_01x02, Connector_PinHeader_2.54mm:PinHeader_1x02_P2.54mm_Horizontal, F.Cu at (184.1, 101.1)
- added J11: Conn_01x02, Connector_PinHeader_2.54mm:PinHeader_1x02_P2.54mm_Horizontal, F.Cu at (184.1, 94.5)
- added J7: Conn_01x06, Connector_JST:JST_XH_S6B-XH-A_1x06_P2.50mm_Horizontal, F.Cu at (185.0, 89.1)
- added J8: Conn_01x02, Connector_PinHeader_2.54mm:PinHeader_1x02_P2.54mm_Horizontal, F.Cu at (176.0, 104.1)
- added J9: Conn_01x02, Connector_PinHeader_2.54mm:PinHeader_1x02_P2.54mm_Horizontal, F.Cu at (169.4, 104.1)
- added R10: 10k, Resistor_SMD:R_0805_2012Metric_Pad1.20x1.40mm_HandSolder, F.Cu at (134.7, 80.7)
- added R11: 10k, Resistor_SMD:R_0805_2012Metric_Pad1.20x1.40mm_HandSolder, F.Cu at (170.9, 97.3)
- added R12: 10k, Resistor_SMD:R_0805_2012Metric_Pad1.20x1.40mm_HandSolder, F.Cu at (179.8, 102.4)
- added R13: 10k, Resistor_SMD:R_0805_2012Metric_Pad1.20x1.40mm_HandSolder, F.Cu at (178.1, 93.7)
- added R14: 10k, Resistor_SMD:R_0805_2012Metric_Pad1.20x1.40mm_HandSolder, F.Cu at (172.0, 100.8)
- added R15: 10k, Resistor_SMD:R_0805_2012Metric_Pad1.20x1.40mm_HandSolder, F.Cu at (179.8, 98.6)
- added R16: 10k, Resistor_SMD:R_0805_2012Metric_Pad1.20x1.40mm_HandSolder, F.Cu at (179.6, 90.2)
- added R7: 5.11k, Resistor_SMD:R_0805_2012Metric_Pad1.20x1.40mm_HandSolder, F.Cu at (132.9, 99.5)
- added R8: 1M, Resistor_SMD:R_0805_2012Metric_Pad1.20x1.40mm_HandSolder, F.Cu at (127.9, 97.9)
- added R9: 5.11k, Resistor_SMD:R_0805_2012Metric_Pad1.20x1.40mm_HandSolder, F.Cu at (132.9, 97.2)
- added U4: AMS1117-3.3, Package_TO_SOT_SMD:SOT-223-3_TabPin2, F.Cu at (148.3, 97.3)
- added U5: NUP4202, Package_TO_SOT_SMD:SOT-363_SC-70-6, F.Cu at (143.5, 79.8)
- added U6: NUP4202, Package_TO_SOT_SMD:SOT-363_SC-70-6, F.Cu at (179.8, 82.8)
- added U7: NUP4202, Package_TO_SOT_SMD:SOT-363_SC-70-6, F.Cu at (141.2, 100.8)
- added U8: NUP4202, Package_TO_SOT_SMD:SOT-363_SC-70-6, F.Cu at (172.0, 79.2)
- added U9: NUP4202, Package_TO_SOT_SMD:SOT-363_SC-70-6, F.Cu at (172.8, 45.6)
- C1, C14: moved to F.Cu
- C10: value 1u -> 10u
- FB1: footprint Resistor_SMD:R_0805_2012Metric_Pad1.20x1.40mm_HandSolder -> Inductor_SMD:L_0805_2012Metric_Pad1.15x1.40mm_HandSolder
- J1: value USB_B_Mini -> USB4105-GF-A; footprint Connector_USB:USB_Mini-B_Lumberg_2486_01_Horizontal -> MyLib:GCT_USB4105-GF-A
- J2, J3, J4, J6: footprint Connector_PinSocket_2.54mm:PinSocket_1x04_P2.54mm_Vertical -> Connector_JST:JST_XH_S4B-XH-A_1x04_P2.50mm_Horizontal
- moved C4 235.1 mm to (279.2, -145.9)
- moved R4 222.7 mm to (286.1, -118.0)
- moved R6 222.7 mm to (286.1, -115.1)
- moved D1 222.7 mm to (280.7, -121.9)
- moved D2 222.7 mm to (280.7, -117.1)
- moved D3 222.7 mm to (286.9, -121.9)
- moved R5 222.7 mm to (292.3, -122.8)
- moved 3v3 184.9 mm to (180.9, -90.8)
- moved C11 184.9 mm to (162.7, -112.4)
- moved C12 184.9 mm to (162.7, -106.7)
- moved C13 184.9 mm to (170.1, -82.6)
- moved C2 184.9 mm to (184.3, -113.1)
- moved C3 184.9 mm to (189.4, -111.2)
- moved C5 184.9 mm to (186.2, -107.4)
- moved C6 184.9 mm to (183.0, -122.6)
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Connections:
- C9 pad 1: (no net) -> unconnected-(C9-Pad1)
- J4 pad 2: /STM32F412/SWDIO -> /STM32F412/CAN_TX
- J4 pad 3: /STM32F412/SWDCLK -> /STM32F412/CAN_RX
- J4 pad 4: (no net) -> GND
- J6 pad 2: /STM32F412/CAN_TX -> /STM32F412/SWDIO
- J6 pad 3: /STM32F412/CAN_RX -> /STM32F412/SWDCLK
- R4 pad 1: (no net) -> unconnected-(R4-Pad1)
- R5 pad 1: (no net) -> unconnected-(R5-Pad1)
- R6 pad 1: (no net) -> unconnected-(R6-Pad1)
- U1 pad 10: (no net) -> /STM32F412/I2S2_ext_SD
- U1 pad 11: (no net) -> /STM32F412/I2S2_SD
- U1 pad 14: (no net) -> /STM32F412/ADC1_IN0
- U1 pad 15: (no net) -> /STM32F412/ADC1_IN1
- U1 pad 16: (no net) -> /STM32F412/ADC1_IN2
- U1 pad 17: (no net) -> /STM32F412/ADC1_IN3
- U1 pad 2: (no net) -> unconnected-(U1-Pad2)
- U1 pad 20: (no net) -> unconnected-(U1-Pad20)
- U1 pad 21: (no net) -> unconnected-(U1-Pad21)
- U1 pad 22: (no net) -> unconnected-(U1-Pad22)
- U1 pad 23: (no net) -> unconnected-(U1-Pad23)
- U1 pad 24: (no net) -> unconnected-(U1-Pad24)
- U1 pad 26: (no net) -> unconnected-(U1-Pad26)
- U1 pad 27: (no net) -> unconnected-(U1-Pad27)
- U1 pad 28: (no net) -> unconnected-(U1-Pad28)
- U1 pad 3: (no net) -> unconnected-(U1-Pad3)
- U1 pad 30: (no net) -> unconnected-(U1-Pad30)
- U1 pad 33: (no net) -> /STM32F412/I2S2_WS
- U1 pad 34: (no net) -> /STM32F412/I2S2_CK
- U1 pad 35: (no net) -> unconnected-(U1-Pad35)
- U1 pad 36: (no net) -> unconnected-(U1-Pad36)
- U1 pad 37: (no net) -> unconnected-(U1-Pad37)
- U1 pad 38: (no net) -> unconnected-(U1-Pad38)
- U1 pad 39: (no net) -> unconnected-(U1-Pad39)
- U1 pad 4: (no net) -> unconnected-(U1-Pad4)
- U1 pad 40: (no net) -> unconnected-(U1-Pad40)
- U1 pad 41: (no net) -> unconnected-(U1-Pad41)
- U1 pad 42: (no net) -> unconnected-(U1-Pad42)
- U1 pad 43: (no net) -> unconnected-(U1-Pad43)
- U1 pad 50: (no net) -> unconnected-(U1-Pad50)
- U1 pad 51: (no net) -> unconnected-(U1-Pad51)
- U1 pad 52: (no net) -> unconnected-(U1-Pad52)
- U1 pad 53: (no net) -> unconnected-(U1-Pad53)
- U1 pad 54: (no net) -> unconnected-(U1-Pad54)
- U1 pad 55: (no net) -> unconnected-(U1-Pad55)
- U1 pad 56: (no net) -> unconnected-(U1-Pad56)
- U1 pad 57: (no net) -> unconnected-(U1-Pad57)
- U1 pad 8: (no net) -> unconnected-(U1-Pad8)
- U1 pad 9: (no net) -> unconnected-(U1-Pad9)
- U2 pad 1: /STM32F412/D+ -> /STM32F412/D-
- U2 pad 3: (no net) -> unconnected-(U2-Pad3)
- U2 pad 4: (no net) -> unconnected-(U2-Pad4)
- U2 pad 6: /STM32F412/D- -> /STM32F412/D+
- U3 pad 6: (no net) -> unconnected-(U3-Pad6)
Routing:
- net /STM32F412/ADC1_IN0: track 0.00 -> 24.1 mm
- net /STM32F412/ADC1_IN2: track 0.00 -> 23.1 mm
- net /STM32F412/ADC1_IN1: track 0.00 -> 19.3 mm
- net /STM32F412/ADC1_IN3: track 0.00 -> 18.2 mm
- net Net-(J1-PadA5): track 0.00 -> 13.3 mm
- net /STM32F412/D-: track 16.9 -> 6.07 mm
- net /STM32F412/D+: track 16.3 -> 6.96 mm
- net /STM32F412/I2S2_SD: track 0.00 -> 8.98 mm
- net /STM32F412/I2S2_CK: track 0.00 -> 8.98 mm
- net Net-(J1-PadB5): track 0.00 -> 8.08 mm
- net /STM32F412/I2S2_ext_SD: track 0.00 -> 7.33 mm
- net /STM32F412/I2S2_WS: track 0.00 -> 7.30 mm
- net Net-(J1-Pad6): track 7.15 -> 0.00 mm, vias 16 -> 0
- net /STM32F412/SWDIO: track 0.00 -> 6.37 mm
- net /STM32F412/SWDCLK: track 0.00 -> 6.34 mm
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Other:
- board size 50.8 x 39.4 mm -> 70 x 50 mm
- net class Default removed
- board text added: "PWR IN"

Commit message: Final layout for V1, sent of to FAB
Parts:
- removed 3v3: TestPoint, TestPoint:TestPoint_Pad_1.0x1.0mm
- removed C14: 100n, Capacitor_SMD:C_0805_2012Metric_Pad1.18x1.45mm_HandSolder
- removed the C9 at (183.4, -94.0)
- removed D1, D2, D3: LED, LED_SMD:LED_PLCC-2
- removed R2, R3, R4, R5, R6: 10k, Resistor_SMD:R_0805_2012Metric_Pad1.20x1.40mm_HandSolder
- removed U3: MS5611-01BA, Package_LGA:LGA-8_3x5mm_P1.25mm
- moved C4 255.8 mm to (152.7, 76.5)
- moved C1 210.7 mm to (160.0, 94.2), turned to -90 degrees
- moved C2 205.9 mm to (163.1, 91.7)
- moved C3 204.9 mm to (148.6, 89.7), turned to 90 degrees
- moved C11 202.1 mm to (166.6, 89.7), turned to 180 degrees
- moved C6 198.8 mm to (162.8, 75.2), turned to 180 degrees
- moved Y1 196.2 mm to (166.8, 86.7), turned to 180 degrees
- moved C12 190.6 mm to (166.6, 83.8), turned to 0 degrees
- moved J5 190.2 mm to (128.0, 75.4), turned to 90 degrees
- moved R1 185.7 mm to (138.7, 82.3)
- moved C5 185.5 mm to (157.7, 75.9)
- moved FB1 183.1 mm to (161.8, 69.6)
- moved C7 173.0 mm to (162.8, 72.1), turned to 180 degrees
- moved C13 168.1 mm to (146.1, 83.8), turned to 180 degrees
- moved C8 163.2 mm to (158.2, 69.6), turned to -90 degrees
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Connections:
- J2 pad 2: /STM32F412/SDA -> /STM32F412/SCL
- J2 pad 3: /STM32F412/SCL -> /STM32F412/SDA
- J4 pad 2: /STM32F412/CAN_TX -> /STM32F412/CAN_RX
- J4 pad 3: /STM32F412/CAN_RX -> /STM32F412/CAN_TX
- J6 pad 2: /STM32F412/SWDIO -> /STM32F412/SWDCLK
- J6 pad 3: /STM32F412/SWDCLK -> /STM32F412/SWDIO
- U5 pad 3: /STM32F412/SWDCLK -> /STM32F412/SWDIO
- U5 pad 4: /STM32F412/SWDIO -> /STM32F412/SWDCLK
- U7 pad 3: /STM32F412/SCL -> /STM32F412/SDA
- U7 pad 4: /STM32F412/SDA -> /STM32F412/SCL
- U9 pad 3: /STM32F412/CAN_RX -> /STM32F412/CAN_TX
- U9 pad 4: /STM32F412/CAN_TX -> /STM32F412/CAN_RX
Routing:
- net +3V3: track 56.9 -> 310.5 mm, vias 0 -> 5
- net GND: track 11.2 -> 123.1 mm, vias 6 -> 54
- net /STM32F412/I2S2_WS: track 7.30 -> 43.9 mm, vias 0 -> 2
- net /STM32F412/I2S2_CK: track 8.98 -> 45.3 mm, vias 0 -> 2
- net /STM32F412/I2S2_ext_SD: track 7.33 -> 32.1 mm, vias 0 -> 2
- net Net-(R1-Pad1): track 0.00 -> 23.3 mm, vias 0 -> 2
- net VBUS: track 6.40 -> 28.7 mm, vias 0 -> 2
- net /STM32F412/SDA: track 6.08 -> 27.5 mm
- net /STM32F412/SCL: track 6.11 -> 27.5 mm
- net /STM32F412/I2S2_SD: track 8.98 -> 30.2 mm, vias 0 -> 2
- net /STM32F412/SWDCLK: track 6.34 -> 25.8 mm
- net /STM32F412/SWDIO: track 6.37 -> 24.9 mm
- net +3.3VA: track 0.00 -> 17.2 mm, vias 0 -> 2
- net Net-(C13-Pad1): track 0.00 -> 16.3 mm, vias 0 -> 2
- net /STM32F412/D+: track 6.96 -> 23.0 mm
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- added copper zone on F.Cu, net +3V3
- added copper zone on B.Cu, net GND
- added copper zone on F.Cu, net GND
- added copper zone on B.Cu, net Net-(J1-PadS1)
- added copper zone on F.Cu, net Net-(J1-PadS1)
Other:
- board text added: "A_0"
- board text added: "A_1"
- board text added: "A_2"
- board text added: "A_3"
- board text added: "CAN"
- board text added: "I2C"
- board text added: "I2S"
- board text added: "SWD"
- board text added: "UART"

Commit message: Update universal.kicad_pcb
Other:
- board text added: "0x00"
- board text added: "SAE 09.2022"
Changed lines of the file:
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@@
   (gr_line (start 125 70) (end 125 110) (layer "Edge.Cuts") (width 0.05))
   (gr_line (start 130 115) (end 190 115) (layer "Edge.Cuts") (width 0.05))
+  (gr_text "SAE\n09.2022" (at 183.134 108.204) (layer "B.SilkS")
+    (effects (font (size 1.5 1) (thickness 0.15)) (justify mirror))
+  )
+  (gr_text "0x00" (at 183.134 111.506) (layer "B.SilkS")
+    (effects (font (size 1.5 1) (thickness 0.15)) (justify mirror))
+  )
   (gr_text "A_1" (at 179.07 112.776) (layer "F.SilkS")
     (effects (font (size 1 1) (thickness 0.15)))
@@
     (effects (font (size 1.5 1) (thickness 0.15)))
   )
+  (gr_text "0x00" (at 183.134 111.506) (layer "F.SilkS")
+    (effects (font (size 1.5 1) (thickness 0.15)))
+  )
   (gr_text "A_2\n" (at 192.532 105.156) (layer "F.SilkS")
     (effects (font (size 1 1) (thickness 0.15)))
@@
     (effects (font (size 1 1) (thickness 0.15)))
   )
+  (gr_text "SAE\n09.2022" (at 183.134 108.204) (layer "F.SilkS")
+    (effects (font (size 1.5 1) (thickness 0.15)))
+  )
   (gr_text "CAN" (at 160.02 101.346) (layer "F.SilkS")
